Commit message: 修改livox启动脚本及增加底盘伺服电机故障读取

File: catkin_ws/src/grinder_gazebo/urdf/x920_grinder.gazebo.xacro (robot description, xacro)
@@ -1,28 +1,40 @@
 <?xml version="1.0"?>
 <robot xmlns:xacro="http://www.ros.org/wiki/xacro">
+  <!-- Damped contacts for the 800 kg body. Very small kd excites numerical
+       chassis oscillation that overwhelms the configurable sensor noise. -->
+  <xacro:macro name="imu_noise_axis" params="axis stddev bias dynamic">
+    <xacro:element xacro:name="${axis}">
+      <noise type="gaussian">
+        <mean>0.0</mean><stddev>${stddev}</stddev>
+        <bias_mean>0.0</bias_mean><bias_stddev>${bias}</bias_stddev>
+        <dynamic_bias_stddev>${dynamic}</dynamic_bias_stddev>
+        <dynamic_bias_correlation_time>${sensor_noise['imu_bias_correlation_time_s']}</dynamic_bias_correlation_time>
+      </noise>
+    </xacro:element>
+  </xacro:macro>
   <gazebo reference="base_link">
     <material>Gazebo/Orange</material>
     <selfCollide>false</selfCollide>
     <!-- Fixed/lumped grinding-disc collision inherits the base contact surface. -->
-    <mu1>0.0</mu1><mu2>0.0</mu2><kp>1000000</kp><kd>10</kd>
+    <mu1>0.0</mu1><mu2>0.0</mu2><kp>1000000</kp><kd>10000</kd>
   </gazebo>
   <gazebo reference="grinding_disc_link">
     <material>Gazebo/Grey</material>
     <!-- The disc and its spherical universal-support contact are frictionless. -->
-    <mu1>0.0</mu1><mu2>0.0</mu2><kp>1000000</kp><kd>10</kd>
+    <mu1>0.0</mu1><mu2>0.0</mu2><kp>1000000</kp><kd>10000</kd>
   </gazebo>
   <gazebo reference="grinding_disc_caster_wheel_link">
     <material>Gazebo/Black</material>
-    <mu1>0.0</mu1><mu2>0.0</mu2><kp>1000000</kp><kd>10</kd>
+    <mu1>0.0</mu1><mu2>0.0</mu2><kp>1000000</kp><kd>10000</kd>
   </gazebo>
   <gazebo reference="left_wheel_link">
     <material>Gazebo/Black</material>
     <!-- Drive wheels retain traction; zero friction here makes diff-drive immobile. -->
-    <mu1>1.0</mu1><mu2>1.0</mu2><kp>1000000</kp><kd>10</kd>
+    <mu1>1.0</mu1><mu2>1.0</mu2><kp>1000000</kp><kd>10000</kd>
   </gazebo>
   <gazebo reference="right_wheel_link">
     <material>Gazebo/Black</material>
     <!-- Drive wheels retain traction; zero friction here makes diff-drive immobile. -->
-    <mu1>1.0</mu1><mu2>1.0</mu2><kp>1000000</kp><kd>10</kd>
+    <mu1>1.0</mu1><mu2>1.0</mu2><kp>1000000</kp><kd>10000</kd>
   </gazebo>
   <gazebo>
@@ -40,8 +52,9 @@
       <commandTopic>$(arg sim_command_topic)</commandTopic>
       <odometryTopic>$(arg sim_odom_topic)</odometryTopic>
-      <odometryFrame>odom</odometryFrame>
-      <robotBaseFrame>base_footprint</robotBaseFrame>
+      <odometryFrame>sim_world</odometryFrame>
+      <robotBaseFrame>base_link</robotBaseFrame>
       <publishWheelTF>false</publishWheelTF>
-      <publishOdomTF>true</publishOdomTF>
+      <!-- Only Super-LIO publishes odom -> base_link. -->
+      <publishOdomTF>false</publishOdomTF>
       <publishWheelJointState>true</publishWheelJointState>
       <odometrySource>world</odometrySource>
@@ -49,22 +62,46 @@
   </gazebo>
   <gazebo reference="laser_link">
-    <sensor type="ray" name="x920_laser">
+    <sensor type="ray" name="mid360s_lidar">
       <always_on>true</always_on>
-      <visualize>true</visualize>
-      <update_rate>15</update_rate>
+      <visualize>false</visualize>
+      <update_rate>10</update_rate>
       <pose>0 0 0 0 0 0</pose>
       <ray>
         <scan>
           <horizontal>
-            <samples>720</samples><resolution>1</resolution>
-            <min_angle>-${pi}</min_angle><max_angle>${pi}</max_angle>
+            <samples>$(arg lidar_horizontal_samples)</samples><resolution>1</resolution>
+            <min_angle>-${pi}</min_angle><max_angle>${pi - 2*pi/int('$(arg lidar_horizontal_samples)')}</max_angle>
           </horizontal>
+          <vertical>
+            <samples>$(arg lidar_vertical_samples)</samples><resolution>1</resolution>
+            <min_angle>${-7*pi/180}</min_angle><max_angle>${52*pi/180}</max_angle>
+          </vertical>
         </scan>
-        <range><min>0.08</min><max>20.0</max><resolution>0.01</resolution></range>
-        <noise><type>gaussian</type><mean>0.0</mean><stddev>0.005</stddev></noise>
+        <range><min>0.10</min><max>$(arg lidar_max_range)</max><resolution>0.01</resolution></range>
+        <noise><type>gaussian</type><mean>0.0</mean><stddev>${sensor_noise['lidar_range_stddev_m']}</stddev></noise>
       </ray>
-      <plugin name="x920_laser_ros" filename="libgazebo_ros_laser.so">
-        <topicName>/scan</topicName>
-        <frameName>laser_link</frameName>
+      <plugin name="mid360s_ros" filename="libgrinder_mid360_sensor.so" />
+    </sensor>
+    <sensor type="imu" name="mid360s_imu">
+      <always_on>true</always_on><update_rate>200</update_rate>
+      <pose>0.011 0.02329 -0.04412 0 0 0</pose>
+      <imu>
+        <angular_velocity>
+          <xacro:imu_noise_axis axis="x" stddev="${sensor_noise['imu_gyro_stddev_rad_s']}" bias="${sensor_noise['imu_gyro_bias_stddev_rad_s']}" dynamic="${sensor_noise['imu_gyro_dynamic_bias_stddev']}" />
+          <xacro:imu_noise_axis axis="y" stddev="${sensor_noise['imu_gyro_stddev_rad_s']}" bias="${sensor_noise['imu_gyro_bias_stddev_rad_s']}" dynamic="${sensor_noise['imu_gyro_dynamic_bias_stddev']}" />
+          <xacro:imu_noise_axis axis="z" stddev="${sensor_noise['imu_gyro_stddev_rad_s']}" bias="${sensor_noise['imu_gyro_bias_stddev_rad_s']}" dynamic="${sensor_noise['imu_gyro_dynamic_bias_stddev']}" />
+        </angular_velocity>
+        <linear_acceleration>
+          <xacro:imu_noise_axis axis="x" stddev="${sensor_noise['imu_accel_stddev_m_s2']}" bias="${sensor_noise['imu_accel_bias_stddev_m_s2']}" dynamic="${sensor_noise['imu_accel_dynamic_bias_stddev']}" />
+          <xacro:imu_noise_axis axis="y" stddev="${sensor_noise['imu_accel_stddev_m_s2']}" bias="${sensor_noise['imu_accel_bias_stddev_m_s2']}" dynamic="${sensor_noise['imu_accel_dynamic_bias_stddev']}" />
+          <xacro:imu_noise_axis axis="z" stddev="${sensor_noise['imu_accel_stddev_m_s2']}" bias="${sensor_noise['imu_accel_bias_stddev_m_s2']}" dynamic="${sensor_noise['imu_accel_dynamic_bias_stddev']}" />
+        </linear_acceleration>
+      </imu>
+      <plugin name="mid360s_imu_ros" filename="libgazebo_ros_imu_sensor.so">
+        <robotNamespace>/</robotNamespace><topicName>/livox/imu</topicName>
+        <frameName>mid360_imu_link</frameName><updateRateHZ>200</updateRateHZ>
+        <!-- Native IMU sensor already applies separate gyro/accel noise and drift. -->
+        <gaussianNoise>0.0</gaussianNoise>
+        <initialOrientationAsReference>false</initialOrientationAsReference>
       </plugin>
     </sensor>

File: catkin_ws/src/grinder_gazebo/urdf/x920_grinder.urdf.xacro (robot description, xacro)
@@ -4,10 +4,21 @@
   <xacro:arg name="visual_mesh" default="false" />
   <xacro:arg name="sim_command_topic" default="/grinder/sim/cmd_vel" />
-  <xacro:arg name="sim_odom_topic" default="/odom" />
+  <xacro:arg name="sim_odom_topic" default="/grinder/sim/ground_truth/odom" />
+  <xacro:arg name="lidar_x" default="0.20" />
+  <xacro:arg name="lidar_y" default="0.0" />
+  <xacro:arg name="lidar_z" default="0.55" />
+  <xacro:arg name="lidar_horizontal_samples" default="360" />
+  <xacro:arg name="lidar_vertical_samples" default="20" />
+  <!-- 仿真最大量程（m），不修改真实 MID-360S 的硬件参数。 -->
+  <xacro:arg name="lidar_max_range" default="45.0" />
+  <xacro:arg name="sensor_noise_config" default="$(find grinder_gazebo)/config/sensor_noise.yaml" />
+  <xacro:property name="sensor_noise" value="${xacro.load_yaml('$(arg sensor_noise_config)')}" />
+  <xacro:property name="lidar_x" value="$(arg lidar_x)" />
+  <xacro:property name="lidar_z" value="$(arg lidar_z)" />
   <!-- Values shared with grinder_chassis_driver/config/chassis_driver.yaml. -->
   <xacro:property name="wheel_track" value="0.70" />
   <xacro:property name="wheel_radius" value="0.1475" />
   <xacro:property name="wheel_width" value="0.10" />
-  <!-- Rear edge is x=-0.30; axle/radar center is 0.30 m forward at x=0.00. -->
+  <!-- Rear drive axle midpoint is the motion reference x=0; lidar is +0.20 m. -->
   <xacro:property name="drive_axle_x" value="0.00" />
   <!-- Exact diff-drive footprint: x=[-0.30, 1.00], y=[-0.47, 0.47]. -->
@@ -26,10 +37,11 @@
   <!-- Front caster contact offset inside the grinding-disc footprint. -->
   <xacro:property name="caster_support_offset_x" value="0.15" />
+  <xacro:property name="caster_radius" value="0.055" />
   <xacro:property name="body_mass" value="${vehicle_mass - disc_mass - caster_mass - 2*drive_wheel_mass - laser_mass - 2*camera_mass}" />
   <!-- This body-link COM makes the complete mass-weighted x COM equal 0.55 m. -->
-  <xacro:property name="body_com_x" value="${(vehicle_mass*0.55 - disc_mass*0.55 - caster_mass*(0.55 + caster_support_offset_x) - 2*camera_mass*0.72) / body_mass}" />
+  <xacro:property name="body_com_x" value="${(vehicle_mass*0.55 - disc_mass*0.55 - caster_mass*(0.55 + caster_support_offset_x) - laser_mass*lidar_x - 2*camera_mass*0.72) / body_mass}" />
   <!-- Put the aggregate COM at the disc centre height as well as its x
        position.  All link origins use base_link at the wheel axle height. -->
-  <xacro:property name="body_com_z" value="${(vehicle_mass*0.04 - disc_mass*0.04 - caster_mass*0.04 - 2*drive_wheel_mass*wheel_radius - laser_mass*(wheel_radius + 0.55) - 2*camera_mass*(wheel_radius + 0.45)) / body_mass - wheel_radius}" />
+  <xacro:property name="body_com_z" value="${(vehicle_mass*0.04 - disc_mass*0.04 - caster_mass*caster_radius - 2*drive_wheel_mass*wheel_radius - laser_mass*(wheel_radius + lidar_z) - 2*camera_mass*(wheel_radius + 0.45)) / body_mass - wheel_radius}" />
   <!-- Place the hidden frictionless caster contact 150 mm ahead of the disc
        centre, still inside its 0.90 m swept footprint.  This gives the rear
@@ -88,7 +100,7 @@
   <link name="base_footprint" />
   <joint name="base_footprint_joint" type="fixed">
-    <parent link="base_footprint" />
-    <child link="base_link" />
-    <origin xyz="0 0 ${wheel_radius}" rpy="0 0 0" />
+    <parent link="base_link" />
+    <child link="base_footprint" />
+    <origin xyz="0 0 ${-wheel_radius}" rpy="0 0 0" />
   </joint>
   <link name="base_link">
@@ -141,8 +153,7 @@
     </inertial>
     <collision name="grinding_disc_caster_collision">
-      <!-- The frictionless front caster carries the remaining front load;
-           its center is set for nominal zero-floor clearance. -->
-      <origin xyz="0 0 0.015" rpy="0 0 0" />
-      <geometry><sphere radius="0.055" /></geometry>
+      <!-- Keep the sphere concentric with the rolling joint. An offset here
+           rotates with the link, changing support height and pitching the body. -->
+      <geometry><sphere radius="${caster_radius}" /></geometry>
     </collision>
   </link>
@@ -153,5 +164,5 @@
     <parent link="base_link" />
     <child link="grinding_disc_caster_wheel_link" />
-    <origin xyz="${0.55 + caster_support_offset_x} 0 -0.1075" rpy="0 0 0" />
+    <origin xyz="${0.55 + caster_support_offset_x} 0 ${caster_radius - wheel_radius}" rpy="0 0 0" />
     <!-- Free rolling axis for the universal support. -->
     <axis xyz="0 1 0" />
@@ -187,5 +198,5 @@
     <xacro:box_inertia mass="${laser_mass}" x="0.08" y="0.08" z="0.06" />
     <visual>
-      <geometry><cylinder radius="0.04" length="0.06" /></geometry>
+      <geometry><box size="0.065 0.065 0.060" /></geometry>
       <material name="sensor_black" />
     </visual>
@@ -195,6 +206,13 @@
     <parent link="base_link" />
     <child link="laser_link" />
-    <!-- Radar is aligned with the two rear drive wheels. -->
-    <origin xyz="${drive_axle_x} 0 0.55" rpy="0 0 0" />
+    <!-- +X is toward the grinding disc; height is relative to the rear axle. -->
+    <origin xyz="$(arg lidar_x) $(arg lidar_y) $(arg lidar_z)" rpy="0 0 0" />
+  </joint>
+  <!-- Match the existing Super-LIO T_imu_laser; this is a simulation convention,
+       not a newly measured MID-360S factory calibration. -->
+  <link name="mid360_imu_link" />
+  <joint name="mid360_imu_joint" type="fixed">
+    <parent link="laser_link" /><child link="mid360_imu_link" />
+    <origin xyz="0.011 0.02329 -0.04412" rpy="0 0 0" />
   </joint>
   <xacro:macro name="camera_link" params="name y">
